File: cbar/cbar.kicad_sch (KiCad schematic)
At the start: 19 parts, among them J1 USB_C_Receptacle_PowerOnly_12V, SW1_PWR SW_SPST, SW2_TILT_SWITCH SW_Push_Shielded, SW3_BATT_IND SW_Push, SW4_SQUISH SW_Push, SW5_DING SW_Push, SW6_WOOSH SW_Push

Commit message: Schematic update
Parts:
- removed SW6_WOOSH: SW_Push, symbol Switch:SW_Push
- added D1: LED1_PLUG_INDICATOR, symbol Device:LED
- added D2: D, symbol Device:D
- added R1: 1kohm, symbol Device:R
- added SW3_TILT_RESET: SW_Push_Shielded, symbol Switch:SW_Push_Shielded
- A1: value RaspberryPi_Pico -> Waveshare RP2040Tiny
- renumbered SW2_TILT_SWITCH to SW2_TILT_TRIGGER, SW4_SQUISH to SW4_METAL, SW5_DING to SW5_MEAT
Connections:
- net 12VGND: now also R1.1
- net 12Vin: now also D2.1 (K); no longer J1.A9 (VBUS), J1.B9 (VBUS)
- net 5VGND: now also U4. (L-), SW3_TILT_RESET.2
- net GP0: now also SW4_METAL.1
- net GP1: now also SW5_MEAT.1
- net GP15: now also SW2_TILT_TRIGGER.1
- net GP4: now also U4. (L-)
- net GP14: now reaches A1.19 (GPIO14)
- net GP14: now also SW3_TILT_RESET.1
- net GP2: no longer names the net of A1.4 (GPIO2)
- new net: D1.2 (A), D2.2 (A), J1.A9 (VBUS), J1.B9 (VBUS)
- new net: D1.1 (K), R1.2
- no-connect marks 0 -> 7
Other:
- moved on the sheet: SW1_PWR, SW4_METAL, SW5_MEAT, U1

Commit message: Schematic update
Parts:
- added D3: D, symbol Device:D
- added R2: 1kohm, symbol Device:R
Connections:
- net 5VGND: now also R2.1
- net GP13: now reaches A1.17 (GPIO13)
- net GP13: now also D3.2 (A)
Changed lines of the file:
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@@
 	)
 	(junction
+		(at 165.1 114.3)
+		(diameter 0)
+		(color 0 0 0 0)
+	)
+	(junction
 		(at 165.1 104.14)
 		(diameter 0)
@@
 	(wire
 		(pts
+			(xy 162.56 114.3) (xy 165.1 114.3)
+		)
+		(stroke
+			(width 0)
+			(type default)
+		)
+	)
+	(wire
+		(pts
 			(xy 81.28 40.64) (xy 90.17 40.64)
 		)
@@
 	(wire
 		(pts
+			(xy 165.1 114.3) (xy 165.1 120.65)
+		)
+		(stroke
+			(width 0)
+			(type default)
+		)
+	)
+	(wire
+		(pts
 			(xy 156.21 80.01) (xy 165.1 80.01)
 		)
@@
 	(wire
 		(pts
+			(xy 165.1 114.3) (xy 165.1 104.14)
+		)
+		(stroke
+			(width 0)
+			(type default)
+		)
+	)
+	(wire
+		(pts
 			(xy 81.28 53.34) (xy 86.36 53.34)
 		)
@@
 		)
 	)
+	(global_label "GP13"
+		(shape input)
+		(at 148.59 114.3 180)
+		(fields_autoplaced yes)
+		(effects
+			(font
+				(size 1.27 1.27)
+			)
+			(justify right)
+		)
+		(property "Intersheetrefs" "${INTERSHEET_REFS}"
+			(at 140.6458 114.3 0)
+			(effects
+				(font
+					(size 1.27 1.27)
+				)
+				(justify right)
+				(hide yes)
+			)
+		)
+	)
 	(global_label "B-"
 		(shape input)
@@
 		)
 	)
+	(global_label "GP13"
+		(shape input)
+		(at 223.52 77.47 180)
+		(fields_autoplaced yes)
+		(effects
+			(font
+				(size 1.27 1.27)
+			)
+			(justify right)
+		)
+		(property "Intersheetrefs" "${INTERSHEET_REFS}"
+			(at 215.5758 77.47 0)
+			(effects
+				(font
+					(size 1.27 1.27)
+				)
+				(justify right)
+				(hide yes)
+			)
+		)
+	)
 	(global_label "GP14"
 		(shape input)
@@
 	)
 	(symbol
+		(lib_id "Device:R")
+		(at 158.75 114.3 270)
+		(unit 1)
+		(exclude_from_sim no)
+		(in_bom yes)
+		(on_board yes)
+		(dnp no)
+		(fields_autoplaced yes)
+		(property "Reference" "R2"
+			(at 158.75 107.95 90)
+			(effects
+				(font
+					(size 1.27 1.27)
+				)
+			)
+		)
+		(property "Value" "1kohm"
+			(at 158.75 110.49 90)
+			(effects
+				(font
+					(size 1.27 1.27)
+				)
+			)
+		)
+		(property "Footprint" ""
+			(at 158.75 112.522 90)
+			(effects
+				(font
+					(size 1.27 1.27)
+				)
+				(hide yes)
+			)
+		)
+		(property "Datasheet" "~"
+			(at 158.75 114.3 0)
+			(effects
+				(font
+					(size 1.27 1.27)
+				)
+				(hide yes)
+			)
+		)
+		(property "Description" "Resistor"
+			(at 158.75 114.3 0)
+			(effects
+				(font
+					(size 1.27 1.27)
+				)
+				(hide yes)
+			)
+		)
+		(pin "2"
+		)
+		(pin "1"
+		)
+		(instances
+			(project "cbar"
+				(path "/32f70377-46f3-4517-9f26-9d1b4abc6052"
+					(reference "R2")
+					(unit 1)
+				)
+			)
+		)
+	)
+	(symbol
 		(lib_id "Device:Speaker")
 		(at 45.72 135.89 0)
@@
 	)
 	(symbol
+		(lib_id "Device:D")
+		(at 152.4 114.3 180)
+		(unit 1)
+		(exclude_from_sim no)
+		(in_bom yes)
+		(on_board yes)
+		(dnp no)
+		(fields_autoplaced yes)
+		(property "Reference" "D3"
+			(at 152.4 107.95 0)
+			(effects
+				(font
+					(size 1.27 1.27)
+				)
+			)
+		)
+		(property "Value" "D"
+			(at 152.4 110.49 0)
+			(effects
+				(font
+					(size 1.27 1.27)
+				)
+			)
+		)
+		(property "Footprint" ""
+			(at 152.4 114.3 0)
+			(effects
+				(font
+					(size 1.27 1.27)
+				)
+				(hide yes)
+			)
+		)
+		(property "Datasheet" "~"
+			(at 152.4 114.3 0)
+			(effects
+				(font
+					(size 1.27 1.27)
+				)
+				(hide yes)
+			)
+		)
+		(property "Description" "Diode"
+			(at 152.4 114.3 0)
+			(effects
+				(font
+					(size 1.27 1.27)
+				)
+				(hide yes)
+			)
+		)
+		(property "Sim.Device" "D"
+			(at 152.4 114.3 0)
+			(effects
+				(font
+					(size 1.27 1.27)
+				)
+				(hide yes)
+			)
+		)
+		(property "Sim.Pins" "1=K 2=A"
+			(at 152.4 114.3 0)
+			(effects
+				(font
+					(size 1.27 1.27)
+				)
+				(hide yes)
+			)
+		)
+		(pin "2"
+		)
+		(pin "1"
+		)
+		(instances
+			(project "cbar"
+				(path "/32f70377-46f3-4517-9f26-9d1b4abc6052"
+					(reference "D3")
+					(unit 1)
+				)
+			)
+		)
+	)
+	(symbol
 		(lib_id "Device:Battery_Cell")
 		(at 86.36 66.04 0)
@@
 	(symbol
 		(lib_id "power:GND")
-		(at 165.1 104.14 0)
+		(at 165.1 120.65 0)
 		(unit 1)
 		(exclude_from_sim no)
@@
 		(fields_autoplaced yes)
 		(property "Reference" "#PWR07"
-			(at 165.1 110.49 0)
+			(at 165.1 127 0)
 			(effects
 				(font
@@
 		)
 		(property "Value" "5VGND"
-			(at 165.1 109.22 0)
+			(at 165.1 125.73 0)
 			(effects
 				(font
@@
 		)
 		(property "Footprint" ""
-			(at 165.1 104.14 0)
+			(at 165.1 120.65 0)
 			(effects
 				(font
@@
 		)
 		(property "Datasheet" ""
-			(at 165.1 104.14 0)
+			(at 165.1 120.65 0)
 			(effects
 				(font
@@
 		)
 		(property "Description" "Power symbol creates a global label with name \"GND\" , ground"
-			(at 165.1 104.14 0)
+			(at 165.1 120.65 0)
 			(effects
 				(font

Commit message: Refactoring
Parts:
- LED2: renamed from D3; value D -> ON INDICATOR (RED)
- R1: value 1kohm -> 9.8kohm
- R2: value 1kohm -> 100 ohm
- renumbered D1 to LED1
Connections:
- net at R2.2: now also LED2.1 (K)
Other:
- moved on the sheet: LED2
Changed lines of the file:
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@@
+	(wire
+		(pts
+			(xy 146.05 114.3) (xy 154.94 114.3)
+		)
+		(stroke
+			(width 0)
+			(type default)
+		)
+	)
 	(wire
 		(pts
@@
 	(global_label "GP13"
 		(shape input)
-		(at 148.59 114.3 180)
+		(at 138.43 114.3 180)
 		(fields_autoplaced yes)
 		(effects
@@
 		)
 		(property "Intersheetrefs" "${INTERSHEET_REFS}"
-			(at 140.6458 114.3 0)
+			(at 130.4858 114.3 0)
 			(effects
 				(font
@@
 			)
 		)
-		(property "Value" "1kohm"
+		(property "Value" "100 ohm"
 			(at 158.75 110.49 90)
 			(effects
@@
 	(symbol
 		(lib_id "Device:D")
-		(at 152.4 114.3 180)
+		(at 142.24 114.3 180)
 		(unit 1)
 		(exclude_from_sim no)
@@
 		(dnp no)
 		(fields_autoplaced yes)
-		(property "Reference" "D3"
-			(at 152.4 107.95 0)
-			(effects
-				(font
-					(size 1.27 1.27)
-				)
-			)
-		)
-		(property "Value" "D"
-			(at 152.4 110.49 0)
+		(property "Reference" "LED2"
+			(at 142.24 107.95 0)
+			(effects
+				(font
+					(size 1.27 1.27)
+				)
+			)
+		)
+		(property "Value" "ON INDICATOR (RED)"
+			(at 142.24 110.49 0)
 			(effects
 				(font
@@
 		)
 		(property "Footprint" ""
-			(at 152.4 114.3 0)
+			(at 142.24 114.3 0)
 			(effects
 				(font
@@
 		)
 		(property "Datasheet" "~"
-			(at 152.4 114.3 0)
+			(at 142.24 114.3 0)
 			(effects
 				(font
@@
 		)
 		(property "Description" "Diode"
-			(at 152.4 114.3 0)
+			(at 142.24 114.3 0)
 			(effects
 				(font
@@
 		)
 		(property "Sim.Device" "D"
-			(at 152.4 114.3 0)
+			(at 142.24 114.3 0)
 			(effects
 				(font
@@
 		)
 		(property "Sim.Pins" "1=K 2=A"
-			(at 152.4 114.3 0)
+			(at 142.24 114.3 0)
 			(effects
 				(font
@@
 			(project "cbar"
 				(path "/32f70377-46f3-4517-9f26-9d1b4abc6052"
-					(reference "D3")
+					(reference "LED2")
 					(unit 1)
 				)
@@
 			)
 		)
-		(property "Value" "1kohm"
+		(property "Value" "9.8kohm"
 			(at 50.8 38.0999 0)
 			(effects
@@
 		(dnp no)
 		(fields_autoplaced yes)
-		(property "Reference" "D1"
+		(property "Reference" "LED1"
 			(at 52.07 29.5274 90)
 			(effects
@@
 			(project ""
 				(path "/32f70377-46f3-4517-9f26-9d1b4abc6052"
-					(reference "D1")
+					(reference "LED1")
 					(unit 1)
 				)
